Commit message: Switched to ignition

File: urdf/model.urdf (robot description, URDF)
Before this commit: robot robot, 5 links, 4 joints
Links:
- removed link chassis
- removed link left_wheel
- removed link right_wheel
- added link base_footprint
- added link left_wheel_link, mass 0.1; collision cylinder length=0.01 radius=0.04; visual cylinder length=0.01 radius=0.04
- added link right_wheel_link, mass 0.1; collision cylinder length=0.01 radius=0.04; visual cylinder length=0.01 radius=0.04
- link base_link: mass None -> 0.4; geometry collision cylinder length=0.16 radius=0.08; visual mesh filename=package://bumblebee/models/meshes/turtle1.dae scale=0.001 0.001 0.001
Joints:
- joint caster_wheel_joint: parent chassis -> base_link
- joint chassis_joint: child chassis -> base_link; parent base_link -> base_footprint
- joint left_wheel_joint: child left_wheel -> left_wheel_link; parent base_link -> base_footprint
- joint right_wheel_joint: child right_wheel -> right_wheel_link; parent base_link -> base_footprint
